File: EMISY/schematic/schematic.kicad_sch (KiCad schematic)
At the start: 6 parts

Commit message: chore
Parts:
- removed BT?: Battery, symbol Device:Battery
- removed SW? (x2): SW_Push, symbol Switch:SW_Push
- removed U?: LTC3525-3.3, Package_TO_SOT_SMD:SOT-363_SC-70-6, symbol Regulator_Switching:LTC3525-3.3
- removed U?: STM32L082CZYx, Package_CSP:ST_WLCSP-49_Die447, symbol MCU_ST_STM32L0:STM32L082CZYx
- removed U?: ICM-20948, Sensor_Motion:InvenSense_QFN-24_3x3mm_P0.4mm, symbol Sensor_Motion:ICM-20948
- added C?: 1µF, symbol Device:C
- added C?: 10 µF, symbol Device:C
- added L?: 10µH, symbol Device:L
- added LR44R (x2): Battery_Cell, symbol Device:Battery_Cell
- added Magnetometer: HMC5883L, HMC5883L, symbol New_Library:HMC5883L
- added Microcontroller: STM32L082CZYx, Package_CSP:ST_WLCSP-49_Die447, symbol MCU_ST_STM32L0:STM32L082CZYx
- added OLED: NHD-2.7-12864WDY3, NHD2712864WDY3, symbol New_Library:NHD-2.7-12864WDY3
- added voltageRegulator: LTC3525-3.3, Package_TO_SOT_SMD:SOT-363_SC-70-6, symbol Regulator_Switching:LTC3525
Connections:
- new net: LR44R.1 (+), LR44R.2 (-)
- new net: L?.2, voltageRegulator.6 (SW)
- new net 3 V: C?.1, L?.1, LR44R.1 (+), voltageRegulator.1 (~{SHDN}), voltageRegulator.3 (VIN)
- new net 3.3 V 140 mA: C?.1, voltageRegulator.4 (VOUT)
- new net Earth: C?.2, C?.2, LR44R.2 (-), voltageRegulator.2 (GND), voltageRegulator.5 (GND)
